File: COMMS/Ground Terminal/Tafiti Ground Comms/Tafiti Ground Comms.kicad_pcb (KiCad board)
At the start: 4 copper layers, 64.5 x 73.6 mm, 65 parts, among them J1 USB_B_Micro, J2 USB_B_Micro, J3 Micro_SD_Card_Det, J4 Conn_01x08_Male, SW1 SW_SPDT, SW2 SW_Push, U1 STM32H743VIT6, U2 AMS1117-3.3, U3 Ai-Thinker-Ra-02, U4 Ai-Thinker-Ra-02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

Commit message: Made minor changes to add mounting holes
Parts:
- added H1: MountingHole, MountingHole:MountingHole_3.2mm_M3, F.Cu at (99.5, 90.6)
- added H2: MountingHole, MountingHole:MountingHole_3.2mm_M3, F.Cu at (152.9, 90.7)
- added H3: MountingHole, MountingHole:MountingHole_3.2mm_M3, F.Cu at (140.3, 153.2)
- added H4: MountingHole, MountingHole:MountingHole_3.2mm_M3, F.Cu at (119.4, 153.4)
- moved G*** 1.12 mm to (133.5, 96.5)
Other:
- board text added: "Onboard Communication System"
- board text removed: "Communication System"

Commit message: Pushed minor changes so as to delete the repo
Other:
- board text added: "Ground Communication Subystem"
- board text removed: "Onboard Communication System"
