File: COMMS/Onboard Terminal/Tafiti Onboard Comms/Tafiti Onboard Comms.kicad_pcb (KiCad board)
At the start: 4 copper layers, 90.2 x 96 mm, 44 parts, among them J1 Micro_SD_Card_Det, J2 Conn_01x08_Male, J3 Conn_02x40_Top_Bottom, SW1 SW_SPDT, SW2 SW_Push, U1 STM32H743VIT6, U2 Ai-Thinker-Ra-02, U3 Ai-Thinker-Ra-02, Y1 32.768KHz, Y2 16MHz

Commit message: Added Lora 3D models as well as Silkscreen
Parts:
- added G***: LOGO, LOGO, F.Cu at (94.2, 119.0)
Routing:
- net Net-(D2-Pad2): track 0.00 -> 1.81 mm
Other:
- board text added: "Ant"
- board text added: "Communication Subsystem"
- board text added: "UHF-Band"

Commit message: Pushed minor changes so as to delete the repo
Parts:
- added H1: MountingHole, MountingHole:MountingHole_3.2mm_M3, F.Cu at (85.9, 57.8)
- added H2: MountingHole, MountingHole:MountingHole_3.2mm_M3, F.Cu at (158.3, 57.8)
- added H3: MountingHole, MountingHole:MountingHole_3.2mm_M3, F.Cu at (85.4, 132.9)
- added H4: MountingHole, MountingHole:MountingHole_3.2mm_M3, F.Cu at (158.9, 132.1)
- moved G*** 68.5 mm to (123.3, 57.0)
- moved J3 0.19 mm to (91.3, 136.3)
Other:
- board text added: "Kenya Space Agency V1.3"
- board text added: "OnBoard Communication Subsystem"
- board text added: "Tafiti Nano-satellite"
