File: COMMS/Onboard Terminal/Tafiti Onboard Comms/Tafiti Onboard Comms.kicad_sch (KiCad schematic)
At the start: 44 parts, among them J1 Micro_SD_Card_Det, J2 Conn_01x08_Male, J3 Conn_02x40_Top_Bottom, SW1 SW_SPDT, SW2 SW_Push, U1 STM32H743VIT6, U2 Ai-Thinker-Ra-02, U3 Ai-Thinker-Ra-02, Y1 32.768KHz, Y2 16MHz

Commit message: Pushed minor changes so as to delete the repo
Parts:
- added H1, H2, H3, H4: MountingHole, symbol Mechanical:MountingHole
Other:
- note added: "Mounting Holes"
